Commit message: [Update][*]修改奖励

File: resources/robots/jump_robot/urdf/jump_robot_qhx_Ori.urdf (robot description, URDF)
Before this commit: robot jump_robot_qhx, 13 links, 12 joints
Links:
- link foot_left: geometry collision mesh filename=../meshes/foot_left.STL; visual mesh filename=../meshes/foot_left.STL
- link foot_right: geometry collision mesh filename=../meshes/foot_right.STL; visual mesh filename=../meshes/foot_right.STL
